File: hardware/tab5_controller/boards/gb/kicad/retropad_gb.kicad_pcb (KiCad board)
At the start: 2 copper layers, 125 x 55 mm, 38 parts, among them J1 Tab5 Ext.Port1, J2 SWD, SW1 UP, SW2 DOWN, SW3 LEFT, SW4 RIGHT, SW5 B, SW6 A, SW7 SELECT, SW8 START, SW9 MENU, U1 STM32F030C8T6

Commit message: tab5_controller: build every console board on the AVR32DD28
The STM32F030 matrix boards are gone. SNES, NES, Game Boy, Genesis and
Master System / Game Gear are now all AVR32DD28 boards: one MCU pin per
button, no diodes, UPDI programming, one firmware image (firmware_avrdd)
keyed by the console-ID straps.

- layout.py / gen_pcb.py / gen_sch.py: drop the stm32 core (LQFP-48,
  key matrix, diodes, SWD header, AN_EN strap); the AVR DD core is the
  only one, and the *_dd board names become the plain console names.
- SNES, NES and Genesis keep the routing of their AVR DD prototypes;
  Game Boy and Master System are routed fresh.
- Every board: DRC 0 unconnected (silkscreen warnings only), schematic
  vs PCB 0 differences, and each switch checked against the MCU pin
  pinmap.h gives it for that console ID.
- Host test now also covers the Game Boy and Master System pin maps.
- READMEs describe the AVR DD boards only.

Co-Authored-By: Claude Opus 5.5 <noreply@anthropic.com>
Claude-Session: https://claude.ai/code/session_01NhSHTsezreiVZCnuBhQzP2
Parts:
- removed C5: 100nF, Capacitor_SMD:C_0603_1608Metric
- removed D1, D2, D3, D4, D5, D6, D7, D8, D9: 1N4148W, Diode_SMD:D_SOD-123
- removed R10: DNP, Resistor_SMD:R_0603_1608Metric
- removed R4, R5: 10k, Resistor_SMD:R_0603_1608Metric
- added R11: DNP, Resistor_SMD:R_0603_1608Metric, B.Cu at (76.0, 93.0)
- J2: value SWD -> UPDI; footprint Connector_PinHeader_2.54mm:PinHeader_1x05_P2.54mm_Vertical -> Connector_PinHeader_2.54mm:PinHeader_1x03_P2.54mm_Vertical
- U1: value STM32F030C8T6 -> AVR32DD28-I/SO; footprint Package_QFP:LQFP-48_7x7mm_P0.5mm -> Package_SO:SOIC-28W_7.5x17.9mm_P1.27mm
- moved R3 17.2 mm to (97.6, 85.7)
- moved C4 12.7 mm to (116.0, 90.5), turned to 90 degrees
- moved C2 11.5 mm to (102.1, 85.7)
- moved C3 7.98 mm to (106.0, 101.6), turned to 180 degrees
- moved C1 5.83 mm to (92.0, 96.0)
- moved J2 2.00 mm to (130.0, 86.5)
- moved R6 2.00 mm to (121.0, 99.0)
- moved R7 2.00 mm to (124.0, 99.0)
- moved R8 2.00 mm to (127.0, 99.0)
- moved R9 2.00 mm to (130.0, 99.0)
- moved U1 0.50 mm to (104.0, 93.5), turned to 90 degrees
Connections:
- J1 pad 10: (no net) -> G9_UPDI
- J1 pad 9: INT -> (no net)
- J2 pad 2: SWCLK -> UPDI
- J2 pad 3: SWDIO -> GND
- R3 pad 2: INT -> RESET
- SW1 pad 2: COL0 -> GND
- SW2 pad 2: COL0 -> GND
- SW3 pad 2: COL0 -> GND
- SW4 pad 2: COL0 -> GND
- SW5 pad 2: COL0 -> GND
- SW6 pad 2: COL0 -> GND
- SW7 pad 2: COL1 -> GND
- SW8 pad 2: COL1 -> GND
- SW9 pad 2: COL2 -> GND
- U1 pad 1: +3V3 -> ID3
- U1 pad 10: COL0 -> K_RIGHT
- U1 pad 11: COL1 -> K_B
- U1 pad 12: COL2 -> K_A
- U1 pad 13: COL3 -> K_SELECT
- U1 pad 14: (no net) -> +3V3
- U1 pad 15: (no net) -> GND
- U1 pad 18: ROW0 -> RESET
- U1 pad 19: ROW1 -> UPDI
- U1 pad 2: (no net) -> K_START
- U1 pad 20: ROW2 -> +3V3
- U1 pad 21: SCL -> GND
- U1 pad 22: SDA -> ID0
- U1 pad 23: GND -> ID1
- U1 pad 24: +3V3 -> SDA
- U1 pad 25: ID0 -> SCL
- U1 pad 26: ID1 -> AN0
- U1 pad 27: ID2 -> AN1
- U1 pad 28: (no net) -> ID2
- U1 pad 3: (no net) -> K_MENU
- U1 pad 6: (no net) -> +3V3
- U1 pad 7: NRST -> K_UP
- U1 pad 8: GND -> K_DOWN
- U1 pad 9: +3V3 -> K_LEFT
Routing:
- net COL0: track 194.4 -> 0.00 mm
- net GND: track 126.8 -> 313.9 mm, vias 2 -> 0
- net ROW0: track 80.5 -> 0.00 mm
- net ROW5: track 64.0 -> 0.00 mm
- net ROW4: track 62.1 -> 0.00 mm
- net ROW2: track 58.4 -> 0.00 mm
- net UPDI: track 0.00 -> 56.5 mm, vias 0 -> 1
- net +3V3: track 97.6 -> 153.0 mm, vias 0 -> 1
- net NRST: track 55.4 -> 0.00 mm, vias 1 -> 0
- net ROW1: track 49.3 -> 0.00 mm
- net COL1: track 47.7 -> 0.00 mm
- net K_A: track 14.6 -> 61.3 mm, vias 0 -> 1
- net K_LEFT: track 9.41 -> 55.1 mm
- net K_DOWN: track 9.41 -> 47.7 mm
- net INT: track 38.2 -> 0.00 mm
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Other:
- board text added: "ID0 ID1 ID2 ID3"
- board text added: "UPDI 3V3 UPDI GND"
- board text removed: "ID0 ID1 ID2 ID3 AN"
- board text removed: "SWD 3V3 CLK DIO RST GND"

Commit message: tab5_controller: remove the UPDI-to-G9 link (R11) from every board
The Tab5 never updates controller firmware, so J1 pin 10 (G9) is left
unconnected, as on M5Stack's keyboard, and R11 and the G9_UPDI net are
gone. Boards are programmed only through their own UPDI header J2.

All five boards are re-routed (the old routes ended at R11). Game Boy
is routed with Freerouting 2.1 single-threaded because 1.9 stalls with
UPDI unrouted on it. Every board: DRC 0 unconnected pads (silkscreen
warnings only), schematic vs PCB 0 differences, switches on the pins
pinmap.h expects.

Co-Authored-By: Claude Opus 5.5 <noreply@anthropic.com>
Claude-Session: https://claude.ai/code/session_01NhSHTsezreiVZCnuBhQzP2
Parts:
- removed R11: DNP, Resistor_SMD:R_0603_1608Metric
Connections:
- J1 pad 10: G9_UPDI -> (no net)
Routing:
- net +3V3: track 153.0 -> 103.9 mm, vias 1 -> 0
- net UPDI: track 56.5 -> 32.1 mm
- net GND: track 313.9 -> 294.5 mm, vias 0 -> 2
- net K_DOWN: track 47.7 -> 63.0 mm, vias 0 -> 1
- net K_SELECT: track 37.1 -> 26.1 mm
- net K_B: track 51.1 -> 59.0 mm
- net G9_UPDI: track 7.36 -> 0.00 mm
- net ID0: track 22.4 -> 26.6 mm
- net K_RIGHT: track 28.1 -> 31.6 mm, vias 0 -> 1
- net ID2: track 19.3 -> 22.4 mm
- net SCL: track 45.0 -> 47.8 mm, vias 0 -> 2
- net K_A: track 61.3 -> 63.8 mm
- net SDA: track 45.4 -> 43.7 mm, vias 0 -> 2
- net K_LEFT: track 55.1 -> 56.7 mm, vias 0 -> 1
- net K_START: track 24.7 -> 26.1 mm
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