File: hardware/tab5_controller/boards/gb/kicad/retropad_gb.kicad_sch (KiCad schematic)
At the start: 46 parts, among them J1 Tab5 Ext.Port1, J2 SWD, SW1 UP, SW10 START, SW11 MENU, SW12 L, SW13 R, SW2 DOWN, SW3 LEFT, SW4 RIGHT, SW5 X, SW6 B, SW7 Y, SW8 A, SW9 SELECT, U1 STM32F030C8T6

Commit message: tab5_controller: NES, Game Boy, Genesis and SMS/GG boards; shared generators
Generators move from boards/snes/kicad to boards/kicad_gen and take a
console name (gen_pcb.py, gen_sch.py, check_netlist.py, plus render.py);
console ids, titles and ID straps come from layout.CONSOLES.

New layouts in layout.py, each passing the clearance checks:
- NES (ID 1): B/A side by side, flat SELECT/START, MENU
- Game Boy (ID 2): diagonal B/A, flat SELECT/START (the angled pair left
  ROW7 unroutable), MENU
- Genesis (ID 5): A/B/C rising row, START, MENU
- Master System / Game Gear (ID 4): 1/2 on the B/A bits, START, MENU

All five boards are regenerated: routed with 0 unconnected pads and no
clearance/edge errors, schematic vs PCB 0 differences, ID straps and
button matrix wiring verified. Connector GND pins and SMD pads now join
the GND pour solidly, which removes starved-thermal errors.

Co-Authored-By: Claude Opus 5.5 <noreply@anthropic.com>
Claude-Session: https://claude.ai/code/session_01NhSHTsezreiVZCnuBhQzP2
Parts:
- removed D10, D11, D12, D13: 1N4148W, Diode_SMD:D_SOD-123, symbol Device:D
- removed SW10: START, Button_Switch_THT:SW_PUSH_6mm, symbol Switch:SW_Push
- removed SW11: MENU, Button_Switch_THT:SW_PUSH_6mm, symbol Switch:SW_Push
- removed SW12: L, Button_Switch_THT:SW_Tactile_SPST_Angled_PTS645Vx31-2LFS, symbol Switch:SW_Push
- removed SW13: R, Button_Switch_THT:SW_Tactile_SPST_Angled_PTS645Vx31-2LFS, symbol Switch:SW_Push
- R6: value 0R -> DNP; now not fitted; now left out of the parts list
- SW5: value X -> B
- SW6: value B -> A
- SW7: value Y -> SELECT; footprint Button_Switch_THT:SW_PUSH-12mm -> Button_Switch_THT:SW_PUSH_6mm
- SW8: value A -> START; footprint Button_Switch_THT:SW_PUSH-12mm -> Button_Switch_THT:SW_PUSH_6mm
- SW9: value SELECT -> MENU
Connections:
- net K_X is gone; now on net K_B: D5.1 (K), SW5.1
- net K_Y is gone; now on net K_SELECT: D7.1 (K), SW7.1
- net COL0: no longer SW8.2
- net COL1: now also SW8.2; no longer SW9.2
- net COL2: now also SW9.2
- net K_A: now also D6.1 (K), SW6.1; no longer D8.1 (K), SW8.1
- net K_B: no longer D6.1 (K), SW6.1
- net K_MENU: now also D9.1 (K), SW9.1
- net K_SELECT: no longer D9.1 (K), SW9.1
- net K_START: now also D8.1 (K), SW8.1
- net ROW0: now also D9.2 (A); no longer D7.2 (A)
- net ROW4: now also D6.2 (A); no longer D8.2 (A)
- net ROW5: now also D5.2 (A); no longer D6.2 (A)
- net ROW6: now also D8.2 (A)
- net ROW7: now also D7.2 (A); no longer D5.2 (A), D9.2 (A)
Other:
- note added: "Console ID straps: 0R to GND = bit set. Game Boy = ID 2 (fit R7; R6, R8, R9, R10 DNP)"
- note removed: "Console ID straps: 0R to GND = bit set. SNES = ID 3 (fit R6, R7; R8, R9, R10 DNP)"
- note removed: "L"
- note removed: "R"
- note removed: "X"
- note removed: "Y"
- title: RetroPad SNES controller (console ID 3) -> RetroPad Game Boy controller (console ID 2)

Commit message: tab5_controller: build every console board on the AVR32DD28
The STM32F030 matrix boards are gone. SNES, NES, Game Boy, Genesis and
Master System / Game Gear are now all AVR32DD28 boards: one MCU pin per
button, no diodes, UPDI programming, one firmware image (firmware_avrdd)
keyed by the console-ID straps.

- layout.py / gen_pcb.py / gen_sch.py: drop the stm32 core (LQFP-48,
  key matrix, diodes, SWD header, AN_EN strap); the AVR DD core is the
  only one, and the *_dd board names become the plain console names.
- SNES, NES and Genesis keep the routing of their AVR DD prototypes;
  Game Boy and Master System are routed fresh.
- Every board: DRC 0 unconnected (silkscreen warnings only), schematic
  vs PCB 0 differences, and each switch checked against the MCU pin
  pinmap.h gives it for that console ID.
- Host test now also covers the Game Boy and Master System pin maps.
- READMEs describe the AVR DD boards only.

Co-Authored-By: Claude Opus 5.5 <noreply@anthropic.com>
Claude-Session: https://claude.ai/code/session_01NhSHTsezreiVZCnuBhQzP2
Parts:
- removed C5: 100nF, Capacitor_SMD:C_0603_1608Metric, symbol Device:C
- removed D1, D2, D3, D4, D5, D6, D7, D8, D9: 1N4148W, Diode_SMD:D_SOD-123, symbol Device:D
- removed R10: DNP, Resistor_SMD:R_0603_1608Metric, symbol Device:R
- removed R4, R5: 10k, Resistor_SMD:R_0603_1608Metric, symbol Device:R
- added R11: DNP, Resistor_SMD:R_0603_1608Metric, symbol Device:R
- J2: value SWD -> UPDI; footprint Connector_PinHeader_2.54mm:PinHeader_1x05_P2.54mm_Vertical -> Connector_PinHeader_2.54mm:PinHeader_1x03_P2.54mm_Vertical; symbol Connector_Generic:Conn_01x05 -> Connector_Generic:Conn_01x03
- U1: value STM32F030C8T6 -> AVR32DD28-I/SO; footprint Package_QFP:LQFP-48_7x7mm_P0.5mm -> Package_SO:SOIC-28W_7.5x17.9mm_P1.27mm; symbol MCU_ST_STM32F0:STM32F030C8Tx -> RetroPad:AVR32DD28-xSO
Connections:
- net COL3 is gone; now on net K_SELECT: U1.13 (PD7)
- net ROW2 is gone; now on net +3V3: U1.20 (VDD)
- net +3V3: now also U1.14 (VDD), U1.6 (VDDIO2); no longer U1.1 (VDD), U1.24 (VDD), U1.48 (VDD), U1.9 (VDDA)
- net GND: now also J2.3 (Pin_3), SW1.2, SW2.2, SW3.2, SW4.2, SW5.2, SW6.2, SW7.2, SW8.2, SW9.2, U1.15 (GND), U1.21 (GND); no longer J2.5 (Pin_5), U1.23 (VSS), U1.47 (VSS), U1.8 (VSSA)
- net ID0: now also U1.22 (XTALHF1/PA0); no longer U1.25 (PB12)
- net ID1: now also U1.23 (XTALHF2/PA1); no longer U1.26 (PB13)
- net ID2: now also U1.28 (PA6); no longer U1.27 (PB14)
- net ID3: now also U1.1 (PA7); no longer U1.45 (PB8)
- net K_A: now also U1.12 (PD6)
- net K_B: now also U1.11 (PD5)
- net K_DOWN: now also U1.8 (PD2)
- net K_LEFT: now also U1.9 (PD3)
- net K_MENU: now also U1.3 (PC1)
- net K_RIGHT: now also U1.10 (PD4)
- net K_START: now also U1.2 (PC0)
- net K_UP: now also U1.7 (PD1)
- net SCL: now also U1.25 (PA3); no longer U1.21 (PB10)
- net SDA: now also U1.24 (PA2); no longer U1.22 (PB11)
- net G9_UPDI: now reaches J1.10 (Pin_10)
- net G9_UPDI: now also R11.2
- removed net AN_EN: U1.46 (PB9)
- removed net BOOT0: U1.44 (BOOT0)
- removed net COL0: SW1.2, SW2.2, SW3.2, SW4.2, SW5.2, SW6.2, U1.10 (PA0)
- removed net COL1: SW7.2, SW8.2, U1.11 (PA1)
- removed net COL2: SW9.2, U1.12 (PA2)
- removed net INT: J1.9 (Pin_9), R3.2, U1.38 (PA15)
- removed net NRST: J2.4 (Pin_4), U1.7 (NRST)
- net ROW0 renamed RESET
- net RESET: now also R3.2
- net ROW1 renamed UPDI
- net UPDI: now also J2.2 (Pin_2), R11.1
- removed net ROW3: U1.39 (PB3)
- removed net ROW4: U1.40 (PB4)
- removed net ROW5: U1.41 (PB5)
- removed net ROW6: U1.42 (PB6)
- removed net ROW7: U1.43 (PB7)
- removed net SWCLK: J2.2 (Pin_2), U1.37 (PA14)
- removed net SWDIO: J2.3 (Pin_3), U1.34 (PA13)
- new net AN0: U1.26 (PA4)
- new net AN1: U1.27 (PA5)
- no-connect marks 20 -> 7
Other:
- note added: "Buttons — one MCU pin each, switch to GND (internal pull-up); slot table in firmware_avrdd/pinmap.h"
- note added: "Console ID straps: 0R to GND = bit set. Game Boy = ID 2 (fit R7; R6, R8, R9 DNP)"
- note added: "Decoupling (VDD x2, VDDIO2), I2C pull-ups, RESET pull-up"
- note added: "MCU — AVR32DD28 (SOIC-28) running firmware_avrdd (I2C client 0x6D, RetroPad protocol)"
- note added: "PD1-PD7, PC0-PC3, PF0-PF1: one button per pin (internal pull-ups)"
- note added: "R11 (DNP): UPDI to J1 pin 10 / G9 — experimental in-system programming from the Tab5"
- note added: "UPDI programming (SerialUPDI / MPLAB Snap)"
- note removed: "Button matrix — row driven high, column read with pull-down; diode anode on the row"
- note removed: "Console ID straps: 0R to GND = bit set. Game Boy = ID 2 (fit R7; R6, R8, R9, R10 DNP)"
- note removed: "Decoupling, pull-ups, reset, BOOT0 (copied from the M5Stack keyboard)"
- note removed: "MCU — STM32F030C8T6 running the RetroPad firmware (I2C slave 0x6D)"
- note removed: "SWD (same order as the keyboard's P2)"
- moved on the sheet: C4, SW1, SW2, SW3, SW4, SW5, SW6, SW7, SW8, SW9

Commit message: tab5_controller: remove the UPDI-to-G9 link (R11) from every board
The Tab5 never updates controller firmware, so J1 pin 10 (G9) is left
unconnected, as on M5Stack's keyboard, and R11 and the G9_UPDI net are
gone. Boards are programmed only through their own UPDI header J2.

All five boards are re-routed (the old routes ended at R11). Game Boy
is routed with Freerouting 2.1 single-threaded because 1.9 stalls with
UPDI unrouted on it. Every board: DRC 0 unconnected pads (silkscreen
warnings only), schematic vs PCB 0 differences, switches on the pins
pinmap.h expects.

Co-Authored-By: Claude Opus 5.5 <noreply@anthropic.com>
Claude-Session: https://claude.ai/code/session_01NhSHTsezreiVZCnuBhQzP2
Parts:
- removed R11: DNP, Resistor_SMD:R_0603_1608Metric, symbol Device:R
Connections:
- net G9_UPDI: no longer names the net of J1.10 (Pin_10)
- no-connect marks 7 -> 8
Other:
- note removed: "R11 (DNP): UPDI to J1 pin 10 / G9 — experimental in-system programming from the Tab5"
Changed lines of the file:
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@@
       (project "retropad_gb" (path "/02035fbd-97ff-5dfe-a404-95c0353b0066" (reference "J1") (unit 1)))))
   (no_connect (at 170.18 39.37))
-  (wire
-    (pts (xy 182.88 49.53) (xy 190.5 49.53))
-    (stroke (width 0) (type default))
-)
-  (global_label
-    "G9_UPDI"
-    (shape bidirectional)
-    (at 190.5 49.53 0)
-    (fields_autoplaced)
-    (effects (font (size 1.27 1.27)) (justify left))
-    (property
-      "Intersheetrefs"
-      "${INTERSHEET_REFS}"
-      (at 190.5 49.53 0)
-      (effects (font (size 1.27 1.27)) hide)))
+  (no_connect (at 182.88 49.53))
   (wire
     (pts (xy 182.88 39.37) (xy 190.5 39.37))
@@
         (path "/02035fbd-97ff-5dfe-a404-95c0353b0066" (reference "#PWR17") (unit 1)))))
   (text
-    "R11 (DNP): UPDI to J1 pin 10 / G9 — experimental in-system programming from the Tab5"
-    (at 150 200 0)
-    (effects (font (size 1.27 1.27)) (justify left))
-)
-  (symbol
-    (lib_id "Device:R")
-    (at 234.95 190.5 0)
-    (unit 1)
-    (in_bom no)
-    (on_board yes)
-    (dnp yes)
-    (property "Reference" "R11" (at 237.49 189.23 0) (effects (font (size 1.27 1.27)) (justify left)))
-    (property "Value" "DNP" (at 237.49 191.77 0) (effects (font (size 1.27 1.27)) (justify left)))
-    (property
-      "Footprint"
-      "Resistor_SMD:R_0603_1608Metric"
-      (at 234.95 190.5 0)
-      (effects (font (size 1.27 1.27)) hide))
-    (property "Datasheet" "~" (at 234.95 190.5 0) (effects (font (size 1.27 1.27)) hide))
-    (pin "1")
-    (pin "2")
-    (instances
-      (project "retropad_gb" (path "/02035fbd-97ff-5dfe-a404-95c0353b0066" (reference "R11") (unit 1)))))
-  (wire
-    (pts (xy 234.95 186.69) (xy 234.95 184.15))
-    (stroke (width 0) (type default))
-)
-  (global_label
-    "UPDI"
-    (shape bidirectional)
-    (at 234.95 184.15 90)
-    (fields_autoplaced)
-    (effects (font (size 1.27 1.27)) (justify left))
-    (property
-      "Intersheetrefs"
-      "${INTERSHEET_REFS}"
-      (at 234.95 184.15 0)
-      (effects (font (size 1.27 1.27)) hide)))
-  (wire
-    (pts (xy 234.95 194.31) (xy 234.95 196.85))
-    (stroke (width 0) (type default))
-)
-  (global_label
-    "G9_UPDI"
-    (shape bidirectional)
-    (at 234.95 196.85 270)
-    (fields_autoplaced)
-    (effects (font (size 1.27 1.27)) (justify right))
-    (property
-      "Intersheetrefs"
-      "${INTERSHEET_REFS}"
-      (at 234.95 196.85 0)
-      (effects (font (size 1.27 1.27)) hide)))
-  (text
     "Mounting holes (M3, 96 mm apart)"
