File: hardware/tab5_controller/boards/genesis/kicad/retropad_genesis.kicad_sch (KiCad schematic)
At the start: 30 parts, among them J1 Tab5 Ext.Port1, J2 UPDI, SW1 UP, SW10 Z, SW11 MODE, SW12 START, SW13 MENU, SW2 DOWN, SW3 LEFT, SW4 RIGHT, SW5 A, SW6 X, SW7 B, SW8 Y, SW9 C, U1 AVR32DD28-I/SO

Commit message: tab5_controller: remove the UPDI-to-G9 link (R11) from every board
The Tab5 never updates controller firmware, so J1 pin 10 (G9) is left
unconnected, as on M5Stack's keyboard, and R11 and the G9_UPDI net are
gone. Boards are programmed only through their own UPDI header J2.

All five boards are re-routed (the old routes ended at R11). Game Boy
is routed with Freerouting 2.1 single-threaded because 1.9 stalls with
UPDI unrouted on it. Every board: DRC 0 unconnected pads (silkscreen
warnings only), schematic vs PCB 0 differences, switches on the pins
pinmap.h expects.

Co-Authored-By: Claude Opus 5.5 <noreply@anthropic.com>
Claude-Session: https://claude.ai/code/session_01NhSHTsezreiVZCnuBhQzP2
Parts:
- removed R11: DNP, Resistor_SMD:R_0603_1608Metric, symbol Device:R
Connections:
- net G9_UPDI: no longer names the net of J1.10 (Pin_10)
- no-connect marks 3 -> 4
Other:
- note removed: "R11 (DNP): UPDI to J1 pin 10 / G9 — experimental in-system programming from the Tab5"
Changed lines of the file:
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@@
         (path "/503e878f-950d-5df8-bd02-9cb70e12f7f1" (reference "J1") (unit 1)))))
   (no_connect (at 170.18 39.37))
-  (wire
-    (pts (xy 182.88 49.53) (xy 190.5 49.53))
-    (stroke (width 0) (type default))
-)
-  (global_label
-    "G9_UPDI"
-    (shape bidirectional)
-    (at 190.5 49.53 0)
-    (fields_autoplaced)
-    (effects (font (size 1.27 1.27)) (justify left))
-    (property
-      "Intersheetrefs"
-      "${INTERSHEET_REFS}"
-      (at 190.5 49.53 0)
-      (effects (font (size 1.27 1.27)) hide)))
+  (no_connect (at 182.88 49.53))
   (wire
     (pts (xy 182.88 39.37) (xy 190.5 39.37))
@@
         (path "/503e878f-950d-5df8-bd02-9cb70e12f7f1" (reference "#PWR17") (unit 1)))))
   (text
-    "R11 (DNP): UPDI to J1 pin 10 / G9 — experimental in-system programming from the Tab5"
-    (at 150 200 0)
-    (effects (font (size 1.27 1.27)) (justify left))
-)
-  (symbol
-    (lib_id "Device:R")
-    (at 234.95 190.5 0)
-    (unit 1)
-    (in_bom no)
-    (on_board yes)
-    (dnp yes)
-    (property "Reference" "R11" (at 237.49 189.23 0) (effects (font (size 1.27 1.27)) (justify left)))
-    (property "Value" "DNP" (at 237.49 191.77 0) (effects (font (size 1.27 1.27)) (justify left)))
-    (property
-      "Footprint"
-      "Resistor_SMD:R_0603_1608Metric"
-      (at 234.95 190.5 0)
-      (effects (font (size 1.27 1.27)) hide))
-    (property "Datasheet" "~" (at 234.95 190.5 0) (effects (font (size 1.27 1.27)) hide))
-    (pin "1")
-    (pin "2")
-    (instances
-      (project
-        "retropad_genesis"
-        (path "/503e878f-950d-5df8-bd02-9cb70e12f7f1" (reference "R11") (unit 1)))))
-  (wire
-    (pts (xy 234.95 186.69) (xy 234.95 184.15))
-    (stroke (width 0) (type default))
-)
-  (global_label
-    "UPDI"
-    (shape bidirectional)
-    (at 234.95 184.15 90)
-    (fields_autoplaced)
-    (effects (font (size 1.27 1.27)) (justify left))
-    (property
-      "Intersheetrefs"
-      "${INTERSHEET_REFS}"
-      (at 234.95 184.15 0)
-      (effects (font (size 1.27 1.27)) hide)))
-  (wire
-    (pts (xy 234.95 194.31) (xy 234.95 196.85))
-    (stroke (width 0) (type default))
-)
-  (global_label
-    "G9_UPDI"
-    (shape bidirectional)
-    (at 234.95 196.85 270)
-    (fields_autoplaced)
-    (effects (font (size 1.27 1.27)) (justify right))
-    (property
-      "Intersheetrefs"
-      "${INTERSHEET_REFS}"
-      (at 234.95 196.85 0)
-      (effects (font (size 1.27 1.27)) hide)))
-  (text
     "Mounting holes (M3, 96 mm apart)"

Commit message: tab5_controller: 0805 hand-solder passives on every board
Swap the 0603 resistors and capacitors (decoupling, I2C pull-ups, reset
pull-up, console-ID straps) for KiCad's 0805 HandSolder footprints, which
have longer pads for soldering by hand. C2 turns 90 degrees so its larger
courtyard clears U1. All four boards are re-routed with Freerouting 1.9;
schematics, BOMs, DRC reports and renders are regenerated.

DRC: 0 errors and 0 unconnected pads on every board (silkscreen and
library-path warnings only). Schematic vs PCB: 0 differences.

Co-Authored-By: Claude Opus 5.5 <noreply@anthropic.com>
Claude-Session: https://claude.ai/code/session_016pgTnJvu7Wh4anaUwDfFmN
Parts:
- C1, C2, C3, C4: footprint Capacitor_SMD:C_0603_1608Metric -> Capacitor_SMD:C_0805_2012Metric_Pad1.18x1.45mm_HandSolder
- R1, R2, R3, R6, R7, R8, R9: footprint Resistor_SMD:R_0603_1608Metric -> Resistor_SMD:R_0805_2012Metric_Pad1.20x1.40mm_HandSolder
Changed lines of the file:
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@@
     (property
       "Footprint"
-      "Capacitor_SMD:C_0603_1608Metric"
+      "Capacitor_SMD:C_0805_2012Metric_Pad1.18x1.45mm_HandSolder"
       (at 160.02 129.54 0)
       (effects (font (size 1.27 1.27)) hide))
@@
     (property
       "Footprint"
-      "Capacitor_SMD:C_0603_1608Metric"
+      "Capacitor_SMD:C_0805_2012Metric_Pad1.18x1.45mm_HandSolder"
       (at 175.26 129.54 0)
       (effects (font (size 1.27 1.27)) hide))
@@
     (property
       "Footprint"
-      "Capacitor_SMD:C_0603_1608Metric"
+      "Capacitor_SMD:C_0805_2012Metric_Pad1.18x1.45mm_HandSolder"
       (at 190.5 129.54 0)
       (effects (font (size 1.27 1.27)) hide))
@@
     (property
       "Footprint"
-      "Capacitor_SMD:C_0603_1608Metric"
+      "Capacitor_SMD:C_0805_2012Metric_Pad1.18x1.45mm_HandSolder"
       (at 204.47 129.54 0)
       (effects (font (size 1.27 1.27)) hide))
@@
     (property
       "Footprint"
-      "Resistor_SMD:R_0603_1608Metric"
+      "Resistor_SMD:R_0805_2012Metric_Pad1.20x1.40mm_HandSolder"
       (at 160.02 154.94 0)
       (effects (font (size 1.27 1.27)) hide))
@@
     (property
       "Footprint"
-      "Resistor_SMD:R_0603_1608Metric"
+      "Resistor_SMD:R_0805_2012Metric_Pad1.20x1.40mm_HandSolder"
       (at 175.26 154.94 0)
       (effects (font (size 1.27 1.27)) hide))
@@
     (property
       "Footprint"
-      "Resistor_SMD:R_0603_1608Metric"
+      "Resistor_SMD:R_0805_2012Metric_Pad1.20x1.40mm_HandSolder"
       (at 190.5 154.94 0)
       (effects (font (size 1.27 1.27)) hide))
@@
     (property
       "Footprint"
-      "Resistor_SMD:R_0603_1608Metric"
+      "Resistor_SMD:R_0805_2012Metric_Pad1.20x1.40mm_HandSolder"
       (at 160.02 190.5 0)
       (effects (font (size 1.27 1.27)) hide))
@@
     (property
       "Footprint"
-      "Resistor_SMD:R_0603_1608Metric"
+      "Resistor_SMD:R_0805_2012Metric_Pad1.20x1.40mm_HandSolder"
       (at 175.26 190.5 0)
       (effects (font (size 1.27 1.27)) hide))
@@
     (property
       "Footprint"
-      "Resistor_SMD:R_0603_1608Metric"
+      "Resistor_SMD:R_0805_2012Metric_Pad1.20x1.40mm_HandSolder"
       (at 190.5 190.5 0)
       (effects (font (size 1.27 1.27)) hide))
@@
     (property
       "Footprint"
-      "Resistor_SMD:R_0603_1608Metric"
+      "Resistor_SMD:R_0805_2012Metric_Pad1.20x1.40mm_HandSolder"
       (at 204.47 190.5 0)
       (effects (font (size 1.27 1.27)) hide))

Commit message: tab5_controller: 4-pin tact switch symbols and footprints
The 6x6 and 12x12 switches are 4-leg parts, and the production layout in
EasyEDA uses their 4-pin symbols, so the KiCad boards now match:

- kicad_lib/RetroPad.pretty: SW_PUSH_6mm_4pin and SW_PUSH-12mm_4pin,
  KiCad's footprints with the pads renumbered 1-4 (pad 1 top-left, then
  clockwise; tied pairs 1-2 and 3-4, the legs 6.5 / 12.5 mm apart).
  gen_pcb.py writes them from the stock footprints and points each
  board's fp-lib-table at the library.
- RetroPad:SW_Push_4pin symbol in gen_sch.py: 1-2 tied, 4-3 tied, one
  contact between. KiCad's 4-pin SW_Push_Dual is a two-contact switch,
  so it doesn't fit these parts.
- Wiring: legs 1-2 to GND, 3-4 to K_<button>. L/R (right angle, two
  contacts plus mounting legs) keep the 2-pin SW_Push.
- All four boards re-routed: DRC 0 unconnected (silkscreen warnings
  only), schematic vs PCB 0 differences, every switch on the pin
  pinmap.h expects; firmware host test passes; Gerber/drill export OK.

Co-Authored-By: Claude Opus 5.5 <noreply@anthropic.com>
Claude-Session: https://claude.ai/code/session_01NhSHTsezreiVZCnuBhQzP2
Parts:
- SW1, SW11, SW12, SW13, SW2, SW3, SW4: footprint Button_Switch_THT:SW_PUSH_6mm -> RetroPad:SW_PUSH_6mm_4pin; symbol Switch:SW_Push -> RetroPad:SW_Push_4pin
- SW10, SW5, SW6, SW7, SW8, SW9: footprint Button_Switch_THT:SW_PUSH-12mm -> RetroPad:SW_PUSH-12mm_4pin; symbol Switch:SW_Push -> RetroPad:SW_Push_4pin
Connections:
- net GND: now also SW1.1, SW10.1, SW11.1, SW12.1, SW13.1, SW2.1, SW3.1, SW4.1, SW5.1, SW6.1, SW7.1, SW8.1, SW9.1
- net K_A: now also SW5.3, SW5.4; no longer SW5.1
- net K_B: now also SW7.3, SW7.4; no longer SW7.1
- net K_C: now also SW9.3, SW9.4; no longer SW9.1
- net K_DOWN: now also SW2.3, SW2.4; no longer SW2.1
- net K_LEFT: now also SW3.3, SW3.4; no longer SW3.1
- net K_MENU: now also SW13.3, SW13.4; no longer SW13.1
- net K_MODE: now also SW11.3, SW11.4; no longer SW11.1
- net K_RIGHT: now also SW4.3, SW4.4; no longer SW4.1
- net K_START: now also SW12.3, SW12.4; no longer SW12.1
- net K_UP: now also SW1.3, SW1.4; no longer SW1.1
- net K_X: now also SW6.3, SW6.4; no longer SW6.1
- net K_Y: now also SW8.3, SW8.4; no longer SW8.1
- net K_Z: now also SW10.3, SW10.4; no longer SW10.1

Commit message: Board schematics: supplies as global labels so EasyEDA keeps GND / +3V3
EasyEDA's KiCad import names a power symbol's net after its library id, so
GND and +3V3 arrived as power_GND and power_+3V3. gen_sch.py now draws every
supply (GND, +3V3, +5V) as a global label, like the other nets. Netlists are
unchanged: GND, +3V3 (+5V on the NES / GB / SMS board), 0 differences vs PCB.

Also:
- pull-up resistor row offset half a pitch so its +3V3 labels clear the
  decoupling capacitors' GND labels
- shorter schematic title so the NES / GB / SMS one fits the title block
- render.py exported the schematic SVG into the folder that also held
  front/back.svg and globbed the first file, so snes and genesis
  schematic.png showed the PCB back view; the schematic now gets its own folder

Co-Authored-By: Claude Opus 5.5 <noreply@anthropic.com>
Claude-Session: https://claude.ai/code/session_01NhSHTsezreiVZCnuBhQzP2
Other:
- title: RetroPad Genesis / Mega Drive 6-button controller (console ID 5) -> RetroPad Genesis / Mega Drive 6-button (console ID 5)
- moved on the sheet: R1, R2, R3
