File: hardware/tab5_controller/boards/nes_gb_sms/kicad/retropad_nes_gb_sms.kicad_pcb (KiCad board)
At the start: 2 copper layers, 125 x 55 mm, 22 parts, among them J1 Tab5 Ext.Port1, J2 UPDI, SW1 UP, SW2 DOWN, SW3 LEFT, SW4 RIGHT, SW5 B, SW6 A, SW7 SELECT, SW8 START, SW9 MENU, U1 AVR32DD28-I/SO

Commit message: NES/GB/SMS board: CONSOLE button + SK6812MINI-E status LED replace the slide switch
Board (nes_gb_sms):
- ID straps now read 14 (SELECT_STRAP_ID), marking a console-select board
- SW_SEL (6x6 tact, front) on PC3; LED1 SK6812MINI-E reverse-mounted on the
  back through a 3.3 x 2.9 mm cutout, datasheet land pattern, data on PC2 via R10
- LED powered from J1 pin 6 (SYS_EXT5V) through D1 1N4148W (~4.3 V, so the
  3.3 V AVR meets the 0.7*VDD input threshold); C5 decoupling
- Track keepout around the cutout; re-routed: 0 unconnected, no copper-edge
  errors, schematic vs PCB 0 differences

Firmware (FW_VERSION 0x22):
- Select mode: console from EEPROM, each debounced press steps NES -> GB -> SMS,
  saved and shown on the LED (red / green / blue); straps not re-read
- Cycle-counted SK6812 bit-bang on VPORTC.2 (1.25 us per bit at 24 MHz)
- Host test covers select mode with a fake EEPROM

Docs: boards, board, firmware and pin-plan READMEs; BOM parts table.

Co-Authored-By: Claude Opus 5.5 <noreply@anthropic.com>
Claude-Session: https://claude.ai/code/session_01NhSHTsezreiVZCnuBhQzP2
Parts:
- removed SW_ID: PCM13SMTR, Button_Switch_SMD:SW_SP3T_PCM13
- added C5: 100nF, Capacitor_SMD:C_0805_2012Metric_Pad1.18x1.45mm_HandSolder, B.Cu at (104.0, 126.5)
- added D1: 1N4148W, Diode_SMD:D_SOD-123, B.Cu at (110.0, 126.5)
- added LED1: SK6812MINI-E, RetroPad:SK6812MINI-E_ReverseMount, B.Cu at (108.0, 131.0)
- added R10: 100, Resistor_SMD:R_0805_2012Metric_Pad1.20x1.40mm_HandSolder, B.Cu at (115.0, 131.0)
- added R6: DNP, Resistor_SMD:R_0805_2012Metric_Pad1.20x1.40mm_HandSolder, B.Cu at (121.0, 99.0)
- added R7: 0R, Resistor_SMD:R_0805_2012Metric_Pad1.20x1.40mm_HandSolder, B.Cu at (124.0, 99.0)
- added R8: 0R, Resistor_SMD:R_0805_2012Metric_Pad1.20x1.40mm_HandSolder, B.Cu at (127.0, 99.0)
- added R9: 0R, Resistor_SMD:R_0805_2012Metric_Pad1.20x1.40mm_HandSolder, B.Cu at (130.0, 99.0)
- added SW_SEL: SELECT CONSOLE, RetroPad:SW_PUSH_6mm_4pin, F.Cu at (94.8, 128.8)
Connections:
- J1 pad 6: (no net) -> +5V
- U1 pad 4: (no net) -> LED_DATA
- U1 pad 5: (no net) -> CON_SEL
Routing:
- net +5V: track 0.00 -> 94.8 mm
- net CON_SEL: track 0.00 -> 47.6 mm
- net LED_DATA: track 0.00 -> 41.3 mm
- net ID0: track 58.5 -> 25.6 mm, vias 1 -> 0
- net ID1: track 54.5 -> 28.3 mm, vias 1 -> 0
- net ID2: track 48.2 -> 23.3 mm, vias 1 -> 0
- net ID3: track 0.00 -> 20.0 mm
- net LED_DIN: track 0.00 -> 19.7 mm
- net +3V3: track 148.0 -> 132.9 mm, vias 0 -> 1
- net K_DOWN: track 50.8 -> 65.6 mm
- net +5V_LED: track 0.00 -> 8.12 mm
- net K_RIGHT: track 30.9 -> 35.5 mm
- net K_UP: track 43.4 -> 40.8 mm, vias 0 -> 1
- net GND: track 307.1 -> 309.6 mm, vias 1 -> 2
- net K_LEFT: track 58.6 -> 56.4 mm, vias 0 -> 1
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Other:
- board text added: "CONSOLE"
- board text added: "ID0"
- board text added: "ID1"
- board text added: "ID2"
- board text added: "ID3"
- board text added: "RetroPad NES / Game Boy / Master System (console IDs 1/2/4)"
- board text removed: "NES GB SMS"
- board text removed: "RetroPad NES / Game Boy / Master System (console ID 1)"

Commit message: Tab5 controller boards: back-side references as board text for EasyEDA
EasyEDA's KiCad import drew the references of R1-R3, R6-R9 and C1-C3
mirrored top to bottom on the back silkscreen, while board-level mirrored
text (ID0-ID3, UPDI labels, board name) came through correctly. Each back
footprint's reference is now redrawn as board text at the same place,
size and angle KiCad shows, and the footprint's own reference is hidden.
KiCad renders are unchanged; DRC counts are unchanged.

Co-Authored-By: Claude Opus 5.5 (1M context) <noreply@anthropic.com>
Claude-Session: https://claude.ai/code/session_01TRQq2EkHCDXMenNyd2D33U
Other:
- board text added: "C1"
- board text added: "C2"
- board text added: "C3"
- board text added: "C4"
- board text added: "C5"
- board text added: "D1"
- board text added: "J2"
- board text added: "LED1"
- board text added: "R1"
- board text added: "R10"
- board text added: "R2"
- board text added: "R3"
- board text added: "R6"
- board text added: "R7"
- board text added: "R8"
- board text added: "R9"
- board text added: "U1"
Changed lines of the file:
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@@
     (property "Sheetname" "")
     (attr smd)
-    (fp_text reference "R8" (at 0 1.65 90) (layer "B.SilkS")
+    (fp_text reference "R8" (at 0 1.65 90) (layer "B.SilkS") hide
         (effects (font (size 1 1) (thickness 0.15)) (justify mirror))
     )
@@
     (property "Sheetname" "")
     (attr smd)
-    (fp_text reference "D1" (at 0 2) (layer "B.SilkS")
+    (fp_text reference "D1" (at 0 2) (layer "B.SilkS") hide
         (effects (font (size 1 1) (thickness 0.15)) (justify mirror))
     )
@@
     (property "Sheetname" "")
     (attr smd)
-    (fp_text reference "R2" (at 0 1.65 90) (layer "B.SilkS")
+    (fp_text reference "R2" (at 0 1.65 90) (layer "B.SilkS") hide
         (effects (font (size 1 1) (thickness 0.15)) (justify mirror))
     )
@@
     (property "Sheetname" "")
     (attr through_hole)
-    (fp_text reference "J2" (at 0 2.33 90) (layer "B.SilkS")
+    (fp_text reference "J2" (at 0 2.33 90) (layer "B.SilkS") hide
         (effects (font (size 1 1) (thickness 0.15)) (justify mirror))
     )
@@
     (property "Sheetname" "")
     (attr smd)
-    (fp_text reference "R7" (at 0 1.65 90) (layer "B.SilkS")
+    (fp_text reference "R7" (at 0 1.65 90) (layer "B.SilkS") hide
         (effects (font (size 1 1) (thickness 0.15)) (justify mirror))
     )
@@
     (property "Sheetname" "")
     (attr smd)
-    (fp_text reference "LED1" (at 0 2.6) (layer "B.SilkS")
+    (fp_text reference "LED1" (at 0 2.6) (layer "B.SilkS") hide
         (effects (font (size 0.8 0.8) (thickness 0.12)) (justify mirror))
     )
@@
     (property "Sheetname" "")
     (attr smd exclude_from_bom)
-    (fp_text reference "R6" (at 0 1.65 90) (layer "B.SilkS")
+    (fp_text reference "R6" (at 0 1.65 90) (layer "B.SilkS") hide
         (effects (font (size 1 1) (thickness 0.15)) (justify mirror))
     )
@@
     (property "Sheetname" "")
     (attr smd)
-    (fp_text reference "C5" (at 0 1.68) (layer "B.SilkS")
+    (fp_text reference "C5" (at 0 1.68) (layer "B.SilkS") hide
         (effects (font (size 1 1) (thickness 0.15)) (justify mirror))
     )
@@
     (property "Sheetname" "")
     (attr smd)
-    (fp_text reference "U1" (at 0 9.9 90) (layer "B.SilkS")
+    (fp_text reference "U1" (at 0 9.9 90) (layer "B.SilkS") hide
         (effects (font (size 1 1) (thickness 0.15)) (justify mirror))
     )
@@
     (property "Sheetname" "")
     (attr smd)
-    (fp_text reference "R1" (at 0 1.65 90) (layer "B.SilkS")
+    (fp_text reference "R1" (at 0 1.65 90) (layer "B.SilkS") hide
         (effects (font (size 1 1) (thickness 0.15)) (justify mirror))
     )
@@
     (property "Sheetname" "")
     (attr smd)
-    (fp_text reference "C4" (at 0 1.68 90) (layer "B.SilkS")
+    (fp_text reference "C4" (at 0 1.68 90) (layer "B.SilkS") hide
         (effects (font (size 1 1) (thickness 0.15)) (justify mirror))
     )
@@
     (property "Sheetname" "")
     (attr smd)
-    (fp_text reference "C2" (at 0 1.68) (layer "B.SilkS")
+    (fp_text reference "C2" (at 0 1.68) (layer "B.SilkS") hide
         (effects (font (size 1 1) (thickness 0.15)) (justify mirror))
     )
@@
     (property "Sheetname" "")
     (attr smd)
-    (fp_text reference "R10" (at 0 1.65 90) (layer "B.SilkS")
+    (fp_text reference "R10" (at 0 1.65 90) (layer "B.SilkS") hide
         (effects (font (size 1 1) (thickness 0.15)) (justify mirror))
     )
@@
     (property "Sheetname" "")
     (attr smd)
-    (fp_text reference "C1" (at 0 1.68 90) (layer "B.SilkS")
+    (fp_text reference "C1" (at 0 1.68 90) (layer "B.SilkS") hide
         (effects (font (size 1 1) (thickness 0.15)) (justify mirror))
     )
@@
     (property "Sheetname" "")
     (attr smd)
-    (fp_text reference "R9" (at 0 1.65 90) (layer "B.SilkS")
+    (fp_text reference "R9" (at 0 1.65 90) (layer "B.SilkS") hide
         (effects (font (size 1 1) (thickness 0.15)) (justify mirror))
     )
@@
     (property "Sheetname" "")
     (attr smd)
-    (fp_text reference "R3" (at 0 1.65 90) (layer "B.SilkS")
+    (fp_text reference "R3" (at 0 1.65 90) (layer "B.SilkS") hide
         (effects (font (size 1 1) (thickness 0.15)) (justify mirror))
     )
@@
     (property "Sheetname" "")
     (attr smd)
-    (fp_text reference "C3" (at 0 1.68) (layer "B.SilkS")
+    (fp_text reference "C3" (at 0 1.68) (layer "B.SilkS") hide
         (effects (font (size 1 1) (thickness 0.15)) (justify mirror))
     )
@@
   (gr_line (start 165 83.5) (end 43 83.5)
     (stroke (width 0.1) (type default)) (layer "Edge.Cuts"))
+  (gr_text "R10" (at 116.65 131 90) (layer "B.SilkS")
+    (effects (font (size 1 1) (thickness 0.15)) (justify mirror))
+  )
+  (gr_text "C1" (at 93.68 96 90) (layer "B.SilkS")
+    (effects (font (size 1 1) (thickness 0.15)) (justify mirror))
+  )
+  (gr_text "R3" (at 99.25 85.7 90) (layer "B.SilkS")
+    (effects (font (size 1 1) (thickness 0.15)) (justify mirror))
+  )
   (gr_text "UPDI 3V3 UPDI GND" (at 132.5 89.4) (layer "B.SilkS")
     (effects (font (size 0.8 0.8) (thickness 0.12)) (justify mirror))
@@
     (effects (font (size 0.8 0.8) (thickness 0.12)) (justify mirror))
   )
+  (gr_text "LED1" (at 108 128.4) (layer "B.SilkS")
+    (effects (font (size 0.8 0.8) (thickness 0.12)) (justify mirror))
+  )
+  (gr_text "R1" (at 87.65 93 90) (layer "B.SilkS")
+    (effects (font (size 1 1) (thickness 0.15)) (justify mirror))
+  )
   (gr_text "ID1" (at 124 102.2) (layer "B.SilkS")
     (effects (font (size 0.8 0.8) (thickness 0.12)) (justify mirror))
   )
+  (gr_text "R8" (at 128.65 99 90) (layer "B.SilkS")
+    (effects (font (size 1 1) (thickness 0.15)) (justify mirror))
+  )
+  (gr_text "R7" (at 125.65 99 90) (layer "B.SilkS")
+    (effects (font (size 1 1) (thickness 0.15)) (justify mirror))
+  )
+  (gr_text "C5" (at 104 124.82) (layer "B.SilkS")
+    (effects (font (size 1 1) (thickness 0.15)) (justify mirror))
+  )
+  (gr_text "R2" (at 85.65 93 90) (layer "B.SilkS")
+    (effects (font (size 1 1) (thickness 0.15)) (justify mirror))
+  )
+  (gr_text "C2" (at 102.1 84.02) (layer "B.SilkS")
+    (effects (font (size 1 1) (thickness 0.15)) (justify mirror))
+  )
+  (gr_text "D1" (at 110 128.5) (layer "B.SilkS")
+    (effects (font (size 1 1) (thickness 0.15)) (justify mirror))
+  )
+  (gr_text "C4" (at 117.68 90.5 90) (layer "B.SilkS")
+    (effects (font (size 1 1) (thickness 0.15)) (justify mirror))
+  )
   (gr_text "ID0" (at 121 102.2) (layer "B.SilkS")
     (effects (font (size 0.8 0.8) (thickness 0.12)) (justify mirror))
   )
+  (gr_text "R6" (at 122.65 99 90) (layer "B.SilkS")
+    (effects (font (size 1 1) (thickness 0.15)) (justify mirror))
+  )
+  (gr_text "J2" (at 132.33 86.5 90) (layer "B.SilkS")
+    (effects (font (size 1 1) (thickness 0.15)) (justify mirror))
+  )
+  (gr_text "U1" (at 113.9 93.5 90) (layer "B.SilkS")
+    (effects (font (size 1 1) (thickness 0.15)) (justify mirror))
+  )
+  (gr_text "C3" (at 106 99.92) (layer "B.SilkS")
+    (effects (font (size 1 1) (thickness 0.15)) (justify mirror))
+  )
+  (gr_text "R9" (at 131.65 99 90) (layer "B.SilkS")
+    (effects (font (size 1 1) (thickness 0.15)) (justify mirror))
+  )
   (gr_text "RetroPad NES_GB_SMS rev 0.1" (at 140 86.5) (layer "B.SilkS")

Commit message: Tab5 controller boards: anchor every footprint on its pad centre for EasyEDA
EasyEDA's KiCad import shifts a footprint whose anchor is off its centre by
the anchor-to-centre distance. On the Genesis board this put the 12 mm
switches on H2 and on R6-R9; J1, J2 and the 6 mm switches were shifted
too. Every footprint now has its anchor on the centre of its pads, in the
routed boards and in the RetroPad switch library, with all pads, tracks
and drawings where they were (checked pad by pad; DRC and netlist
unchanged). --back-refs-only becomes --easyeda-fixups, which applies both
EasyEDA changes to a routed board.

Co-Authored-By: Claude Opus 5.5 (1M context) <noreply@anthropic.com>
Claude-Session: https://claude.ai/code/session_01TRQq2EkHCDXMenNyd2D33U
Parts:
- moved SW5 6.73 mm to (130.0, 118.0)
- moved SW6 6.73 mm to (146.0, 114.0)
- moved J1 5.24 mm to (66.0, 88.8)
- moved SW1 3.95 mm to (70.0, 101.8)
- moved SW2 3.95 mm to (70.0, 126.5)
- moved SW3 3.95 mm to (57.5, 114.0)
- moved SW4 3.95 mm to (82.5, 114.0)
- moved SW7 3.95 mm to (97.8, 119.0)
- moved SW8 3.95 mm to (110.2, 119.0)
- moved SW_SEL 3.95 mm to (98.0, 131.0)
- moved SW9 3.95 mm to (104.0, 109.0)
- moved J2 2.54 mm to (127.5, 86.5)
